File: LaserActive-CU-CLD085-Remote.kicad_pcb (KiCad board)
At the start: 2 copper layers, 36.9 x 119.9 mm, 35 parts, among them IC1 D6600CS, K0 Button, K1 Button, K10 Button, K11 Button, K12 Button, K16 Button, K18 Button, K19 Button, K2 Button, K20 Button, K24 Button, K25 Button, K26 Button, K27 Button, K28 Button, K29 Button, K3 Button, K32 Button, K33 Button, K34 Button, K35 Button, K36 Button, K4 Button, K7 Button, Q1 NPN, X1 Crystal

Commit message: Updates
Connections:
- K0 pad 1: unconnected-(K0-Pad1) -> ROW_6
- K0 pad 2: unconnected-(K0-Pad2) -> ROW_1
- K1 pad 1: unconnected-(K1-Pad1) -> ROW_2
- K1 pad 2: unconnected-(K1-Pad2) -> ROW_6
- K10 pad 1: unconnected-(K10-Pad1) -> ROW_5
- K10 pad 2: ROW_2 -> COL_4
- K11 pad 1: unconnected-(K11-Pad1) -> COL_3
- K11 pad 2: unconnected-(K11-Pad2) -> ROW_5
- K12 pad 1: unconnected-(K12-Pad1) -> ROW_5
- K12 pad 2: unconnected-(K12-Pad2) -> COL_2
- K16 pad 1: COL_1 -> ROW_4
- K18 pad 1: COL_1 -> ROW_4
- K18 pad 2: ROW_2 -> COL_4
- K19 pad 1: COL_1 -> ROW_4
- K19 pad 2: unconnected-(K19-Pad2) -> COL_3
- K2 pad 1: unconnected-(K2-Pad1) -> COL_4
- K2 pad 2: unconnected-(K2-Pad2) -> ROW_6
- K20 pad 1: COL_1 -> ROW_4
- K20 pad 2: unconnected-(K20-Pad2) -> COL_2
- K3 pad 1: unconnected-(K3-Pad1) -> COL_3
- K3 pad 2: unconnected-(K3-Pad2) -> ROW_6
- K4 pad 1: unconnected-(K4-Pad1) -> ROW_6
- K4 pad 2: unconnected-(K4-Pad2) -> COL_2
Routing:
- net unconnected-(D1-A-Pad1): track 0.00 -> 105.6 mm
- net ROW_7: track 0.00 -> 102.9 mm, vias 0 -> 1
- net ROW_2: track 30.5 -> 115.6 mm, vias 0 -> 3
- net COL_4: track 0.00 -> 60.7 mm, vias 0 -> 2
- net ROW_1: track 21.9 -> 79.5 mm, vias 0 -> 2
- net ROW_6: track 0.00 -> 41.3 mm, vias 0 -> 2
- added copper zone on B.Cu, net COL_2
- added copper zone on B.Cu, net COL_3
- added copper zone on B.Cu, net COL_4
- added copper zone on B.Cu, net ROW_4
- added copper zone on B.Cu, net ROW_5
- added copper zone on B.Cu, net ROW_6
- removed copper zone on B.Cu, net (none)
- removed copper zone on B.Cu, net COL_1

Commit message: Update LaserActive-CU-CLD085-Remote.kicad_pcb
Routing:
- added copper zone on B.Cu, net (none)
Changed lines of the file:
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@@
 	(gr_poly
 		(pts
+			(xy 141.5 106.56) (xy 143.53 106.56) (xy 143.53 103.72) (xy 144.75 102.5) (xy 144.75 101.91) (xy 136.02 101.91)
+			(xy 135.18 102.75) (xy 135.18 104.55) (xy 141.58 104.55) (xy 141.58 106.03) (xy 141.44 106.03) (xy 141.44 106.5)
+		)
+		(stroke
+			(width 0)
+			(type solid)
+		)
+		(fill yes)
+		(layer "B.Mask")
+	)
+	(gr_poly
+		(pts
 			(xy 141.46 87.987254) (xy 141.62 87.987254) (xy 141.62 86.557254) (xy 135.1 86.557254) (xy 135.1 84.867254)
 			(xy 136.07 83.897254) (xy 152.11 83.897254) (xy 155.46 87.247254) (xy 155.46 88.027254) (xy 154.98 88.507254)
@@
 	)
 	(zone
+		(net 12)
+		(net_name "ROW_1")
+		(layer "B.Cu")
+		(hatch edge 0.5)
+		(priority 12)
+		(connect_pads yes
+			(clearance 0.1)
+		)
+		(min_thickness 0.1)
+		(filled_areas_thickness no)
+		(fill yes
+			(thermal_gap 0.5)
+			(thermal_bridge_width 0.5)
+			(island_removal_mode 1)
+			(island_area_min 10)
+		)
+		(polygon
+			(pts
+				(xy 154.45 102.37) (xy 155.96 100.86) (xy 156.96 100.86) (xy 157.92 101.82) (xy 166.85 101.82) (xy 167.34 102.31)
+				(xy 167.34 105.5) (xy 166.26 106.58) (xy 165.15 106.58) (xy 165.15 106.05) (xy 165.16 106.04) (xy 165.46 106.04)
+				(xy 165.46 104.54) (xy 159.05 104.54) (xy 159.05 104.02) (xy 156.29 104.02) (xy 155.4 104.91) (xy 155.4 106.54)
+				(xy 153.16 106.54) (xy 153.09 106.47) (xy 153.09 106.07) (xy 153.16 106) (xy 153.61 106) (xy 153.61 104.49)
+				(xy 147.18 104.49) (xy 147.18 103.24) (xy 148.05 102.37)
+			)
+		)
+	)
+	(zone
 		(net 20)
 		(net_name "COL_2")
@@
 	)
 	(zone
+		(net 0)
+		(net_name "")
+		(layer "B.Cu")
+		(hatch edge 0.5)
+		(priority 13)
+		(connect_pads yes
+			(clearance 0.1)
+		)
+		(min_thickness 0.1)
+		(filled_areas_thickness no)
+		(fill yes
+			(thermal_gap 0.5)
+			(thermal_bridge_width 0.5)
+			(island_removal_mode 1)
+			(island_area_min 10)
+		)
+		(polygon
+			(pts
+				(xy 158.68 105.09) (xy 156.78 105.09) (xy 156.29 105.58) (xy 156.29 106.99) (xy 159.08 109.78) (xy 164.51 109.78)
+				(xy 165.02 109.27) (xy 165.02 107.08) (xy 158.55 107.08) (xy 158.55 105.41) (xy 158.68 105.28)
+			)
+		)
+	)
+	(zone
 		(net 15)
 		(net_name "ROW_5")
@@
 			)
 		)
+	)
+	(zone
+		(net 0)
+		(net_name "")
+		(layer "B.Cu")
+		(hatch edge 0.5)
+		(priority 11)
+		(connect_pads yes
+			(clearance 0.1)
+		)
+		(min_thickness 0.1)
+		(filled_areas_thickness no)
+		(fill yes
+			(thermal_gap 0.5)
+			(thermal_bridge_width 0.5)
+			(island_removal_mode 1)
+			(island_area_min 10)
+		)
+		(polygon
+			(pts
+				(xy 141.5 106.56) (xy 143.53 106.56) (xy 143.53 103.72) (xy 144.75 102.5) (xy 144.75 101.91) (xy 136.02 101.91)
+				(xy 135.18 102.75) (xy 135.18 104.55) (xy 141.58 104.55) (xy 141.58 106.03) (xy 141.44 106.03) (xy 141.44 106.5)
+			)
+		)
+	)
+	(zone
+		(net 0)
+		(net_name "")
+		(layer "B.Cu")
+		(hatch edge 0.5)
+		(priority 14)
+		(connect_pads yes
+			(clearance 0.1)
+		)
+		(min_thickness 0.1)
+		(filled_areas_thickness no)
+		(fill yes
+			(thermal_gap 0.5)
+			(thermal_bridge_width 0.5)
+			(island_removal_mode 1)
+			(island_area_min 10)
+		)
+		(polygon
+			(pts
+				(xy 135.14 105.07) (xy 133.14 105.07) (xy 132.7 105.51) (xy 132.7 108.89) (xy 133.13 109.32) (xy 140.77 109.32)
+				(xy 144.54 113.09) (xy 147.09 113.09) (xy 147.09 113.59) (xy 153.57 113.59) (xy 153.57 115.07) (xy 153.42 115.07)
+				(xy 153.39 115.1) (xy 153.39 115.61) (xy 154.06 115.61) (xy 154.06 117.22) (xy 159.25 122.41) (xy 165.6 122.41)
+				(xy 165.6 124.06) (xy 165.4 124.06) (xy 165.23 124.23) (xy 165.23 124.6) (xy 166.91 124.6) (xy 167.4 124.11)
+				(xy 167.4 120.62) (xy 167.13 120.35) (xy 159.68 120.35) (xy 155.54 116.21) (xy 155.54 111.94) (xy 155.08 111.48)
+				(xy 146.16 111.48) (xy 142.27 107.59) (xy 141.03 107.59) (xy 141.03 107.08) (xy 134.7 107.08) (xy 134.7 105.45)
+				(xy 134.86 105.29) (xy 134.92 105.29)
+			)
+		)
