File: LaserActive-CU-CLD085-Remote.kicad_pcb (KiCad board)
At the start: 2 copper layers, 36.9 x 119.9 mm, 35 parts, among them IC1 D6600CS, K0 Button, K1 Button, K10 Button, K11 Button, K12 Button, K16 Button, K18 Button, K19 Button, K2 Button, K20 Button, K24 Button, K25 Button, K26 Button, K27 Button, K28 Button, K29 Button, K3 Button, K32 Button, K33 Button, K34 Button, K35 Button, K36 Button, K4 Button, K7 Button, Q1 NPN, X1 Crystal

Commit message: Update LaserActive-CU-CLD085-Remote.kicad_pcb
Routing:
- net COL_3: track 0.00 -> 43.2 mm, vias 0 -> 1
Changed lines of the file:
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@@
+	)
+	(segment
+		(start 155.98 62.736511)
+		(end 155.98 64.23)
+		(width 0.2)
+		(layer "F.Cu")
+		(net 17)
+	)
+	(segment
+		(start 154.65 93.09)
+		(end 154.65 98.68)
+		(width 0.2)
+		(layer "F.Cu")
+		(net 17)
+	)
+	(segment
+		(start 153.39 82.34)
+		(end 153.39 84.38)
+		(width 0.2)
+		(layer "F.Cu")
+		(net 17)
+	)
+	(segment
+		(start 155.14 65.07)
+		(end 155.14 80.59)
+		(width 0.2)
+		(layer "F.Cu")
+		(net 17)
+	)
+	(segment
+		(start 154.65 98.68)
+		(end 153.43 99.9)
+		(width 0.2)
+		(layer "F.Cu")
+		(net 17)
+	)
+	(segment
+		(start 155.98 64.23)
+		(end 155.14 65.07)
+		(width 0.2)
+		(layer "F.Cu")
+		(net 17)
+	)
+	(segment
+		(start 153.43 99.9)
+		(end 149.86 99.9)
+		(width 0.2)
+		(layer "F.Cu")
+		(net 17)
+	)
+	(segment
+		(start 155.14 80.59)
+		(end 153.39 82.34)
+		(width 0.2)
+		(layer "F.Cu")
+		(net 17)
+	)
+	(segment
+		(start 153.39 84.38)
+		(end 155.12 86.11)
+		(width 0.2)
+		(layer "F.Cu")
+		(net 17)
+	)
+	(segment
+		(start 155.12 92.62)
+		(end 154.65 93.09)
+		(width 0.2)
+		(layer "F.Cu")
+		(net 17)
+	)
+	(segment
+		(start 155.12 86.11)
+		(end 155.12 92.62)
+		(width 0.2)
+		(layer "F.Cu")
+		(net 17)
+	)
+	(via
+		(at 149.86 99.9)
+		(size 0.8)
+		(drill 0.3)
+		(layers "F.Cu" "B.Cu")
+		(net 17)
 	)
 	(segment

Commit message: Updates
Parts:
- C4: footprint Capacitor_THT:CP_Radial_D5.0mm_P2.00mm -> Pioneer:Electrolytic_P2.50mm
- Q1: footprint Package_TO_SOT_THT:TO-220-3_Vertical -> Pioneer:TO-220-3
- X1: footprint Crystal:Crystal_HC18-U_Vertical -> Pioneer:Crystal
- moved C4 0.19 mm to (164.8, 47.5)
Routing:
- net COL_2: track 0.00 -> 96.8 mm, vias 0 -> 5
- net COL_1: track 0.00 -> 85.3 mm, vias 0 -> 1
- net ROW_3: track 0.00 -> 81.7 mm, vias 0 -> 4
- net Net-(IC1-S-IN): track 0.00 -> 70.9 mm, vias 0 -> 2
- net unconnected-(D1-K-Pad3): track 0.00 -> 58.4 mm, vias 0 -> 1
- net ROW_5: track 0.00 -> 53.1 mm, vias 0 -> 3
- net (no net): track 0.00 -> 52.8 mm, vias 0 -> 2
- net COL_3: track 43.2 -> 67.9 mm, vias 1 -> 2
- net ROW_4: track 0.00 -> 22.4 mm, vias 0 -> 1
- net ROW_6: track 41.3 -> 54.2 mm, vias 2 -> 3
- added copper zone on B.Cu, net ROW_3
Other:
- board text added: "B"
- board text added: "E"
