File: LaserActive-CU-CLD085-Remote.kicad_pcb (KiCad board)
At the start: 2 copper layers, 36.9 x 119.9 mm, 37 parts, among them IC1 D6600CS, K0 Button, K1 Button, K10 Button, K11 Button, K12 Button, K16 Button, K18 Button, K19 Button, K2 Button, K20 Button, K24 Button, K25 Button, K26 Button, K27 Button, K28 Button, K29 Button, K3 Button, K32 Button, K33 Button, K34 Button, K35 Button, K36 Button, K4 Button, K7 Button, Q1 NPN, T1 B+, T2 B-, X1 Crystal

Commit message: Updates
Parts:
- moved D3 2.44 mm to (148.7, 50.8), turned to 0 degrees
Connections:
- Q1 pad 1: Net-(D3-A) -> Net-(IC1-REM)
- Q1 pad 2: Net-(IC1-REM) -> Net-(D3-A)
Routing:
- net VCC: track 0.00 -> 203.8 mm
- net GND: track 0.00 -> 176.5 mm
- net Net-(IC1-REM): track 0.00 -> 23.4 mm
- net Net-(D1-A): track 105.6 -> 108.7 mm
- added copper zone on F.Cu, net GND
- added copper zone on B.Cu, net Net-(D3-A)
- added copper zone on B.Cu, net Net-(D3-K)
- added copper zone on F.Cu, net VCC
- removed copper zone on B.Cu, net ROW_5

Commit message: Fix Schematic Values and symbols
Parts:
- C2, C3: value 10pF -> 100pF
- C5: value C_Small -> 100nF
- D1: value D_Dual_CommonAnode_AKK -> DAP215
- Q1: value NPN -> 2SC4037 NPN
- R1: value 220 -> 2.2ohm
- X1: value Crystal -> CSB 480E
Changed lines of the file:
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@@
 	(net 4 "Net-(IC1-OSC-IN)")
 	(net 5 "VCC")
-	(net 6 "Net-(D1-A)")
+	(net 6 "Net-(IC1-S-IN)")
 	(net 7 "COL_6")
 	(net 8 "Net-(D3-K)")
@@
 		)
 		(property "Value" "47uF"
-			(at 1.25 3.5 90)
+			(at 5.5754 0.057324 180)
 			(layer "F.Fab")
 			(effects
@@
 			)
 		)
-		(property "Datasheet" "~"
+		(property "Datasheet" ""
 			(at 0 0 90)
 			(layer "F.Fab")
@@
 			)
 		)
-		(property "Value" "D_Dual_CommonAnode_AKK"
+		(property "Value" "DAP215"
 			(at 2.28 2.2 90)
 			(layer "F.Fab")
@@
 			)
 		)
-		(property "Datasheet" "~"
+		(property "Datasheet" ""
 			(at 0 0 90)
 			(layer "F.Fab")
@@
 			(layers "*.Cu" "*.Mask")
 			(remove_unused_layers no)
-			(net 6 "Net-(D1-A)")
-			(pinfunction "A")
+			(net 6 "Net-(IC1-S-IN)")
+			(pinfunction "K")
 			(pintype "passive")
 		)
@@
 			(remove_unused_layers no)
 			(net 15 "ROW_6")
-			(pinfunction "K")
+			(pinfunction "A")
 			(pintype "passive")
 		)
@@
 			)
 		)
-		(property "Datasheet" "~"
+		(property "Datasheet" ""
 			(at 0 0 0)
 			(unlocked yes)
@@
 			)
 		)
-		(property "Datasheet" "~"
+		(property "Datasheet" ""
 			(at 0 0 0)
 			(unlocked yes)
@@
 			)
 		)
-		(property "Value" "220"
-			(at 2.54 1.92 90)
+		(property "Value" "2.2ohm"
+			(at -3.799287 -0.003916 180)
 			(layer "F.Fab")
 			(effects
@@
 			)
 		)
-		(property "Datasheet" "~"
+		(property "Datasheet" ""
 			(at 0 0 90)
 			(layer "F.Fab")
@@
 			)
 		)
-		(property "Datasheet" "~"
+		(property "Datasheet" ""
 			(at 0 0 0)
 			(unlocked yes)
@@
 			)
 		)
-		(property "Datasheet" "~"
+		(property "Datasheet" ""
 			(at 0 0 0)
 			(layer "F.Fab")
@@
 			)
 		)
-		(property "Datasheet" "~"
+		(property "Datasheet" ""
 			(at 0 0 0)
 			(unlocked yes)
@@
 			)
 		)
-		(property "Datasheet" "~"
+		(property "Datasheet" ""
 			(at 0 0 0)
 			(layer "F.Fab")
@@
 			)
 		)
-		(property "Datasheet" "~"
+		(property "Datasheet" ""
 			(at 0 0 180)
 			(unlocked yes)
@@
 			)
 		)
-		(property "Datasheet" "~"
+		(property "Datasheet" ""
 			(at 0 0 0)
 			(unlocked yes)
@@
 			)
 		)
-		(property "Datasheet" "~"
+		(property "Datasheet" ""
 			(at 0 0 0)
 			(unlocked yes)
@@
 			)
 		)
-		(property "Value" "10pF"
-			(at 8.033016 0.895138 0)
+		(property "Value" "100pF"
+			(at -5.669116 -0.7946 0)
 			(layer "F.Fab")
 			(effects
@@
 			)
 		)
-		(property "Datasheet" "~"
+		(property "Datasheet" ""
 			(at 0 0 0)
 			(layer "F.Fab")
@@
 			)
 		)
-		(property "Datasheet" "~"
+		(property "Datasheet" ""
 			(at 0 0 0)
 			(unlocked yes)
@@
 			)
 		)
-		(property "Datasheet" "~"
+		(property "Datasheet" ""
 			(at 0 0 0)
 			(unlocked yes)
@@
 		(tags "TO-220-3 Vertical RM 2.54mm")
 		(property "Reference" "Q1"
-			(at 2.606215 2.768912 180)
+			(at 2.606215 2.768912 0)
 			(layer "F.SilkS")
 			(effects
@@
 			)
 		)
-		(property "Value" "NPN"
-			(at -0.743352 2.217483 270)
+		(property "Value" "2SC4037 NPN"
+			(at 2.837035 -4.002488 90)
 			(layer "F.Fab")
 			(effects
@@
 		)
 		(property "Datasheet" ""
-			(at 0 0 270)
+			(at 0 0 90)
 			(layer "F.Fab")
 			(hide yes)
@@
 		)
 		(property "Description" ""
-			(at 0 0 270)
+			(at 0 0 90)
 			(layer "F.Fab")
 			(hide yes)
@@
 			)
 		)
+		(property ki_fp_filters "TO?126*")
 		(sheetname "/")
 		(sheetfile "LaserActive-CU-CLD085-Remote.kicad_sch")
@@
 		)
 		(fp_text user "${REFERENCE}"
-			(at 2.54 -0.95 270)
+			(at 2.54 -0.95 90)
 			(layer "F.Fab")
 			(effects
@@
 			(remove_unused_layers no)
 			(net 17 "Net-(IC1-REM)")
-			(pinfunction "C")
-			(pintype "open_collector")
+			(pinfunction "E")
+			(pintype "passive")
 		)
 		(pad "2" thru_hole oval
@@
 			(remove_unused_layers no)
 			(net 9 "Net-(D3-A)")
-			(pinfunction "B")
-			(pintype "input")
+			(pinfunction "C")
+			(pintype "passive")
 		)
 		(pad "3" thru_hole oval
@@
 			(remove_unused_layers no)
 			(net 2 "GND")
-			(pinfunction "E")
-			(pintype "open_emitter")
+			(pinfunction "B")
+			(pintype "input")
 		)
 		(embedded_fonts no)
@@
 			)
 		)
-		(property "Value" "Crystal"
-			(at 2.45 3.52 0)
+		(property "Value" "CSB 480E"
+			(at 8.1682 1.6604 0)
 			(layer "F.Fab")
 			(effects
@@
 			)
 		)
-		(property "Datasheet" "~"
+		(property "Datasheet" ""
 			(at 0 0 0)
 			(layer "F.Fab")
@@
 			)
 		)
-		(property "Datasheet" "~"
+		(property "Datasheet" ""
 			(at 0 0 0)
 			(unlocked yes)
@@
 		)
 		(property "Value" "IRL81A"
-			(at 1.27 1.86 0)
+			(at 1.2362 -1.8696 0)
 			(layer "F.Fab")
 			(effects
@@
 			)
 		)
-		(property "Value" "10pF"
-			(at 7.606433 1.175037 0)
+		(property "Value" "100pF"
+			(at -5.644856 -1.0278 0)
 			(layer "F.Fab")
 			(effects
@@
 			)
 		)
-		(property "Datasheet" "~"
+		(property "Datasheet" ""
 			(at 0 0 0)
 			(layer "F.Fab")
@@
 			)
 		)
-		(property "Value" "C_Small"
+		(property "Value" "100nF"
 			(at 2.5 -1.931123 90)
 			(layer "F.Fab")
@@
 			)
 		)
-		(property "Datasheet" "~"
+		(property "Datasheet" ""
 			(at 0 0 90)
 			(layer "F.Fab")
@@
 			)
 		)
-		(property "Datasheet" "~"
+		(property "Datasheet" ""
 			(at 0 0 0)
 			(unlocked yes)
@@
 			)
 		)
-		(property "Datasheet" "~"
+		(property "Datasheet" ""
 			(at 0 0 0)
 			(unlocked yes)
@@
 			)
 		)
-		(property "Datasheet" "~"
+		(property "Datasheet" ""
 			(at 0 0 0)
 			(layer "F.Fab")
@@
 			)
 		)
-		(property "Datasheet" "~"
+		(property "Datasheet" ""
 			(at 0 0 0)
 			(unlocked yes)
@@
 			)
 		)
-		(property "Datasheet" "~"
+		(property "Datasheet" ""
 			(at 0 0 0)
 			(unlocked yes)
@@
 			)
 		)
-		(property "Datasheet" "~"
+		(property "Datasheet" ""
 			(at 0 0 0)
 			(unlocked yes)
@@
 			)
 		)
-		(property "Datasheet" "~"
+		(property "Datasheet" ""
 			(at 0 0 180)
 			(unlocked yes)
@@
 		)
 		(property "Value" "D6600CS"
-			(at 3.81 25.19 90)
+			(at 3.81 -2.4578 90)
 			(layer "F.Fab")
 			(effects
@@
 			(layers "*.Cu" "*.Mask")
 			(remove_unused_layers no)
-			(net 6 "Net-(D1-A)")
+			(net 6 "Net-(IC1-S-IN)")
 			(pinfunction "S-IN")
 			(pintype "input")
@@
 			)
 		)
-		(property "Datasheet" "~"
+		(property "Datasheet" ""
 			(at 0 0 0)
 			(unlocked yes)
@@
 			)
 		)
-		(property "Datasheet" "~"
+		(property "Datasheet" ""
 			(at 0 0 0)
 			(unlocked yes)
@@
 			)
 		)
-		(property "Datasheet" "~"
+		(property "Datasheet" ""
 			(at 0 0 0)
 			(unlocked yes)
@@
 			)
 		)
-		(property "Datasheet" "~"
+		(property "Datasheet" ""
 			(at 0 0 0)
 			(unlocked yes)
@@
 			)
 		)
-		(property "Datasheet" "~"
+		(property "Datasheet" ""
 			(at 0 0 0)
 			(unlocked yes)
@@
 			)
 		)
-		(property "Datasheet" "~"
+		(property "Datasheet" ""
 			(at 0 0 180)
 			(unlocked yes)
@@
 			)
 		)
-		(property "Datasheet" "~"
+		(property "Datasheet" ""
 			(at 0 0 180)
 			(unlocked yes)
@@
 			)
 		)
-		(property "Datasheet" "~"
+		(property "Datasheet" ""
 			(at 0 0 0)
 			(unlocked yes)
