File: LaserActive-CU-CLD085-Remote.kicad_sch (KiCad schematic)
At the start: 37 parts, among them IC1 D6600CS, K0 Button, K1 Button, K10 Button, K11 Button, K12 Button, K16 Button, K18 Button, K19 Button, K2 Button, K20 Button, K24 Button, K25 Button, K26 Button, K27 Button, K28 Button, K29 Button, K3 Button, K32 Button, K33 Button, K34 Button, K35 Button, K36 Button, K4 Button, K7 Button, Q1 2SC4037 NPN, T1 B+, T2 B-, X1 CSB 480E

Commit message: Updates
Parts:
- T1, T2: footprint Connector_PinHeader_2.54mm:PinHeader_1x01_P2.54mm_Vertical -> Pioneer:Battery Terminal
Changed lines of the file:
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@@
 			)
 		)
-		(property "Footprint" "Connector_PinHeader_2.54mm:PinHeader_1x01_P2.54mm_Vertical"
+		(property "Footprint" "Pioneer:Battery Terminal"
 			(at 242.57 69.85 0)
 			(effects
@@
 			)
 		)
-		(property "Footprint" "Connector_PinHeader_2.54mm:PinHeader_1x01_P2.54mm_Vertical"
+		(property "Footprint" "Pioneer:Battery Terminal"
 			(at 242.57 78.74 0)
 			(effects

Commit message: Silk Tweaks
Other:
- company: (none) -> Board Folk
- title: (none) -> Laser Active CU-CLD085 Remote Control
Changed lines of the file:
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@@
 	(generator_version "9.0")
 	(paper "A4")
+	(title_block
+		(title "Laser Active CU-CLD085 Remote Control")
+		(date "2026-01-18")
+		(rev "1.0")
+		(company "Board Folk")
+	)
 	(junction
 		(at 158.75 147.32)
