File: LaserActive-CU-CLD085-Remote.kicad_sch (KiCad schematic)
At the start: 37 parts, among them IC1 D6600CS, K0 Button, K1 Button, K10 Button, K11 Button, K12 Button, K16 Button, K18 Button, K19 Button, K2 Button, K20 Button, K24 Button, K25 Button, K26 Button, K27 Button, K28 Button, K29 Button, K3 Button, K32 Button, K33 Button, K34 Button, K35 Button, K36 Button, K4 Button, K7 Button, Q1 2SC4037 NPN, T1 B+, T2 B-, X1 CSB 480E

Commit message: Merged from Zaxour
Parts:
- added C6, C7: 100pF, Capacitor_SMD:C_0603_1608Metric, symbol Device:C_Small
- added C8, C9: 0.1u, Capacitor_SMD:C_0603_1608Metric, symbol Device:C_Small
Connections:
- net GND: now also C6.1, C7.1, C8.1, C9.1
- net VCC: now also C9.2
- net at C2.2, IC1.8 (OSC-IN), X1.1: now also C7.2
- net at C3.2, IC1.7 (OSC-OUT), X1.2: now also C6.2
- net at C1.1, IC1.10 (AC): now also C8.2
Other:
- note added: "C1,C2,C3,C5 THT C6,C7,C8,C9 SMD One or the other"
